Commit message: Add files via upload

File: mobilerobot/urdf/mobilerobot.xacro (robot description, xacro)
@@ -1,130 +1,107 @@
 <?xml version="1.0"?>
-<robot xmlns:xacro="http://www.ros.org/wiki/xacro">
-    <material name="red">
-        <color rgba="1 0 0 1"/>
-    </material>
-    <material name="green">
-        <color rgba="0 1 0 1"/>
-    </material>
-    <material name="blue">
-        <color rgba="0 0 1 1"/>
-    </material>
-    <material name="yellow">
-        <color rgba="1 1 0 1"/>
-    </material>
-     <!---base link -->
-    <link name="base_link"/>
-    <!--chassis link-->
-    <joint name="chassis_joint" type="fixed">
-        <parent link="base_link"/>
-        <child link="chassis"/>
-        <origin xyz="-0.1 0 0" rpy="0 0 0"/>
-    </joint>
-    <link name="chassis">
-        <visual>
-            <origin xyz="0.15 0 0.075" rpy="0 0 0"/>
-            <geometry>
-                <box size="0.35 0.25 0.15"/>
-            </geometry>
-            <material name="blue"/>
-        </visual>
-        <collision>
-            <origin xyz="0.15 0 0.075" rpy="0 0 0"/>
-            <geometry>
-                <box size="0.35 0.25 0.15"/>
-            </geometry>
-        </collision>
-        <inertial>
-            <mass value="2.0"/>
-            <origin xyz="0.15 0 0.075" rpy="0 0 0"/>
-            <inertia ixx="0.01" ixy="0.0" ixz="0.0"
-                     iyy="0.01" iyz="0.0"
-                     izz="0.01"/>
-        </inertial>
-    </link>
-    <!--left wheel link-->
-    <joint name="left_wheel_joint" type="continuous">
-        <parent link="chassis"/>
-        <child link="left_wheel"/>
-        <origin xyz="0.1 0.140 0" rpy="-${pi/2} 0 0"/>
-        <axis xyz="0 0 1"/>
-    </joint>
-    <link name="left_wheel">
-        <visual>
-            <geometry>
-                <cylinder radius="0.06" length="0.03"/>
-            </geometry>
-            <material name="red"/>
-        </visual>
-        <collision>
-            <geometry>
-                <cylinder radius="0.06" length="0.03"/>
-            </geometry>
-        </collision>
-        <inertial>
-            <mass value="0.2"/>
-            <origin xyz="0 0 0" rpy="0 0 0"/>
-            <inertia ixx="0.0001" ixy="0.0" ixz="0.0"
-                     iyy="0.0001" iyz="0.0"
-                     izz="0.0001"/>
-        </inertial>
-    </link>
-    <!--right wheel link-->
-    <joint name="right_wheel_joint" type="continuous">
-        <parent link="chassis"/>
-        <child link="right_wheel"/>
-        <origin xyz="0.1 -0.140 0" rpy="${pi/2} 0 0"/>
-        <axis xyz="0 0 -1"/>
-    </joint>
-    <link name="right_wheel">
-        <visual>
-            <geometry>
-                <cylinder radius="0.06" length="0.03"/>
-            </geometry>
-            <material name="green"/>
-        </visual>
-        <collision>
-            <geometry>
-                <cylinder radius="0.06" length="0.03"/>
-            </geometry>
-        </collision>
-        <inertial>
-            <mass value="0.2"/>
-            <origin xyz="0 0 0" rpy="0 0 0"/>
-            <inertia ixx="0.0001" ixy="0.0" ixz="0.0"
-                     iyy="0.0001" iyz="0.0"
-                     izz="0.0001"/>
-        </inertial>
-    </link>
-    <!--caster link-->
-    <joint name="left_caster_joint" type="fixed">
-        <parent link="chassis"/>
-        <child link="caster"/>
-        <origin xyz="0.24 0 0"/>
-    </joint>
-    <link name="caster">
-        <visual>
-            <geometry>
-                <sphere radius="0.04"/>
-            </geometry>
-            <material name="yellow"/>
-        </visual>
-        <collision>
-            <geometry>
-                <sphere radius="0.04"/>
-            </geometry>
-        </collision>
-        <inertial>
-            <mass value="0.05"/>
-            <origin xyz="0 0 0" rpy="0 0 0"/>
-            <inertia ixx="0.00001" ixy="0.0" ixz="0.0"
-                     iyy="0.00001" iyz="0.0"
-                     izz="0.00001"/>
-        </inertial>
-    </link>
-    <gazebo reference="caster">
-        <material>Gazebo/black</material>
-        <mu1 value="0.001"/>
-        <mu2 value="0.001"/>
-    </gazebo>
+<robot xmlns:xacro="http://www.ros.org/wiki/xacro" name="mobilebot">
+  <!-- Materials -->
+  <material name="red"><color rgba="1 0 0 1"/></material>
+  <material name="green"><color rgba="0 1 0 1"/></material>
+  <material name="blue"><color rgba="0 0 1 1"/></material>
+  <material name="yellow"><color rgba="1 1 0 1"/></material>
+  <material name="black"><color rgba="0 0 0 1"/></material>
+  <!-- Base -->
+  <link name="base_link"/>
+  <!-- Chassis -->
+  <joint name="chassis_joint" type="fixed">
+    <parent link="base_link"/>
+    <child link="chassis"/>
+    <origin xyz="-0.1 0 0" rpy="0 0 0"/>
+  </joint>
+  <link name="chassis">
+    <visual>
+      <origin xyz="0.15 0 0.075" rpy="0 0 0"/>
+      <geometry><box size="0.35 0.25 0.15"/></geometry>
+      <material name="blue"/>
+    </visual>
+    <collision>
+      <origin xyz="0.15 0 0.075" rpy="0 0 0"/>
+      <geometry><box size="0.35 0.25 0.15"/></geometry>
+    </collision>
+    <inertial>
+      <mass value="2.0"/>
+      <origin xyz="0.15 0 0.075" rpy="0 0 0"/>
+      <inertia ixx="0.01" ixy="0" ixz="0" iyy="0.01" iyz="0" izz="0.01"/>
+    </inertial>
+  </link>
+  <!-- Left wheel -->
+  <joint name="left_wheel_joint" type="continuous">
+    <parent link="chassis"/>
+    <child link="left_wheel"/>
+    <origin xyz="0.1 0.140 0" rpy="-${pi/2} 0 0"/>
+    <axis xyz="0 0 1"/>
+  </joint>
+  <link name="left_wheel">
+    <visual><geometry><cylinder radius="0.06" length="0.03"/></geometry><material name="red"/></visual>
+    <collision><geometry><cylinder radius="0.06" length="0.03"/></geometry></collision>
+    <inertial>
+      <mass value="0.2"/><origin xyz="0 0 0"/><inertia ixx="0.0001" ixy="0" ixz="0" iyy="0.0001" iyz="0" izz="0.0001"/>
+    </inertial>
+  </link>
+  <!-- Right wheel -->
+  <joint name="right_wheel_joint" type="continuous">
+    <parent link="chassis"/><child link="right_wheel"/>
+    <origin xyz="0.1 -0.140 0" rpy="${pi/2} 0 0"/>
+    <axis xyz="0 0 -1"/>
+  </joint>
+  <link name="right_wheel">
+    <visual><geometry><cylinder radius="0.06" length="0.03"/></geometry><material name="green"/></visual>
+    <collision><geometry><cylinder radius="0.06" length="0.03"/></geometry></collision>
+    <inertial>
+      <mass value="0.2"/><origin xyz="0 0 0"/><inertia ixx="0.0001" ixy="0" ixz="0" iyy="0.0001" iyz="0" izz="0.0001"/>
+    </inertial>
+  </link>
+  <!-- Caster -->
+  <joint name="left_caster_joint" type="fixed">
+    <parent link="chassis"/><child link="caster"/><origin xyz="0.24 0 0"/>
+  </joint>
+  <link name="caster">
+    <visual><geometry><sphere radius="0.05"/></geometry><material name="yellow"/></visual>
+    <collision><geometry><sphere radius="0.05"/></geometry></collision>
+    <inertial>
+      <mass value="0.05"/><origin xyz="0 0 0"/><inertia ixx="1e-5" ixy="0" ixz="0" iyy="1e-5" iyz="0" izz="1e-5"/>
+    </inertial>
+  </link>
+  <gazebo reference="caster">
+    <material>Gazebo/black</material><mu1 value="0.001"/><mu2 value="0.001"/>
+  </gazebo>
+  <!-- Front camera (box touching front face, centered) -->
+  <!-- Chassis front face is at x = 0.15 + 0.35/2 = 0.325 -->
+  <joint name="front_camera_joint" type="fixed">
+    <parent link="chassis"/><child link="front_camera_link"/>
+    <origin xyz="0.325 0 0.075" rpy="0 0 0"/>
+  </joint>
+  <link name="front_camera_link">
+    <visual><geometry><box size="0.08 0.06 0.06"/></geometry><material name="red"/></visual>
+    <collision><geometry><box size="0.08 0.06 0.06"/></geometry></collision>
+    <inertial>
+      <mass value="0.08"/><origin xyz="0 0 0"/><inertia ixx="5e-5" ixy="0" ixz="0" iyy="5e-5" iyz="0" izz="5e-5"/>
+    </inertial>
+  </link>
+  <!-- Gazebo camera sensor + ROS2 plugin (shows frustum and publishes image) -->
+  <gazebo reference="front_camera_link">
+    <sensor name="front_camera" type="camera">
+      <update_rate>30</update_rate>
+      <visualize>true</visualize> <!-- frustum in Gazebo -->
+      <camera>
+        <horizontal_fov>1.0472</horizontal_fov> <!-- ~60 deg -->
+        <image><width>640</width><height>480</height><format>R8G8B8</format></image>
+        <clip><near>0.05</near><far>50</far></clip>
+      </camera>
+      <plugin name="gazebo_ros_camera" filename="libgazebo_ros_camera.so">
+        <ros>
+          <namespace>/</namespace>
+          <remapping>image_raw:=/front_camera/image_raw</remapping>
+          <remapping>camera_info:=/front_camera/camera_info</remapping>
+        </ros>
+        <frame_name>front_camera_link</frame_name>
+      </plugin>
+    </sensor>
+  </gazebo>
 </robot>
